File: FeedbackSchematic/FeedbackSchematic.kicad_pcb (KiCad board)
At the start: 2 copper layers, 102 parts, among them J1 Screw_Terminal_01x02, J10 Conn_01x02_Male, J11 Conn_01x02_Male, J2 Screw_Terminal_01x08, J3 Conn_01x08_Male, J4 Conn_01x08_Male, J5 Conn_01x08_Male, J6 RJ45, J7 RJ45, J8 Conn_01x04_Male, J9 Conn_01x03_Male, U1 BluePill_STM32F103C, U2 L7805, U3 L7805, U4 6N137, U5 6N137, U6 TJA1050_Board, U7 74HC595, U8 74HC595

Commit message: Latest changes railcom and pcb
Parts:
- moved R3 137.6 mm to (40.6, 25.4), turned to 180 degrees
- moved D2 126.1 mm to (35.6, 20.3)
- moved R2 122.5 mm to (63.5, 27.9)
- moved D1 84.3 mm to (50.8, 15.2), turned to 180 degrees
- moved D31 58.6 mm to (43.2, 76.2)
- moved D22 58.2 mm to (53.3, 30.5), turned to 180 degrees
- moved D32 44.7 mm to (57.9, 70.9), turned to 180 degrees
- moved R63 10.1 mm to (177.8, 109.2)
- moved D21 9.16 mm to (38.1, 35.6)
Changed lines of the file:
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@@
   )
   (footprint "Resistor_THT:R_Axial_DIN0204_L3.6mm_D1.6mm_P5.08mm_Horizontal" (layer "F.Cu")
-    (at 140.890225 119.71)
+    (at 40.64 25.4 180)
     (descr "Resistor, Axial_DIN0204 series, Axial, Horizontal, pin pitch=5.08mm, 0.167W, length*diameter=3.6*1.6mm^2, http://cdn-reichelt.de/documents/datenblatt/B400/1_4W%23YAG.pdf")
     (tags "Resistor Axial_DIN0204 series Axial Horizontal pin pitch 5.08mm 0.167W length 3.6mm diameter 1.6mm")
@@
     (fp_line (start 4.34 -0.8) (end 0.74 -0.8) (layer "F.Fab") (width 0.1))
     (fp_line (start 0.74 0.8) (end 4.34 0.8) (layer "F.Fab") (width 0.1))
-    (pad "1" thru_hole circle (at 0 0) (size 1.4 1.4) (drill 0.7) (layers *.Cu *.Mask)
+    (pad "1" thru_hole circle (at 0 0 180) (size 1.4 1.4) (drill 0.7) (layers *.Cu *.Mask)
       (net 2 "Dcc2") (pintype "passive"))
-    (pad "2" thru_hole oval (at 5.08 0) (size 1.4 1.4) (drill 0.7) (layers *.Cu *.Mask)
+    (pad "2" thru_hole oval (at 5.08 0 180) (size 1.4 1.4) (drill 0.7) (layers *.Cu *.Mask)
       (net 7 "Net-(D1-Pad2)") (pintype "passive"))
     (model "${KICAD6_3DMODEL_DIR}/Resistor_THT.3dshapes/R_Axial_DIN0204_L3.6mm_D1.6mm_P5.08mm_Horizontal.wrl"
@@
   )
   (footprint "Resistor_THT:R_Axial_DIN0204_L3.6mm_D1.6mm_P5.08mm_Horizontal" (layer "F.Cu")
-    (at 140.890225 122.86)
+    (at 63.5 27.94)
     (descr "Resistor, Axial_DIN0204 series, Axial, Horizontal, pin pitch=5.08mm, 0.167W, length*diameter=3.6*1.6mm^2, http://cdn-reichelt.de/documents/datenblatt/B400/1_4W%23YAG.pdf")
     (tags "Resistor Axial_DIN0204 series Axial Horizontal pin pitch 5.08mm 0.167W length 3.6mm diameter 1.6mm")
@@
   )
   (footprint "Resistor_THT:R_Axial_DIN0204_L3.6mm_D1.6mm_P1.90mm_Vertical" (layer "F.Cu")
-    (at 175.760225 99.3)
+    (at 177.8 109.22)
     (descr "Resistor, Axial_DIN0204 series, Axial, Vertical, pin pitch=1.9mm, 0.167W, length*diameter=3.6*1.6mm^2, http://cdn-reichelt.de/documents/datenblatt/B400/1_4W%23YAG.pdf")
     (tags "Resistor Axial_DIN0204 series Axial Vertical pin pitch 1.9mm 0.167W length 3.6mm diameter 1.6mm")
@@
   )
   (footprint "Diode_THT:D_DO-201AD_P15.24mm_Horizontal" (layer "F.Cu")
-    (at 97.020225 92.51)
+    (at 57.919775 70.92 180)
     (descr "Diode, DO-201AD series, Axial, Horizontal, pin pitch=15.24mm, , length*diameter=9.5*5.2mm^2, , http://www.diodes.com/_files/packages/DO-201AD.pdf")
     (tags "Diode DO-201AD series Axial Horizontal pin pitch 15.24mm  length 9.5mm diameter 5.2mm")
@@
     (fp_line (start 12.37 2.6) (end 12.37 -2.6) (layer "F.Fab") (width 0.1))
     (fp_line (start 4.295 -2.6) (end 4.295 2.6) (layer "F.Fab") (width 0.1))
-    (pad "1" thru_hole rect (at 0 0) (size 3.2 3.2) (drill 1.6) (layers *.Cu *.Mask)
+    (pad "1" thru_hole rect (at 0 0 180) (size 3.2 3.2) (drill 1.6) (layers *.Cu *.Mask)
       (net 7 "Net-(D1-Pad2)") (pinfunction "K") (pintype "passive"))
-    (pad "2" thru_hole oval (at 15.24 0) (size 3.2 3.2) (drill 1.6) (layers *.Cu *.Mask)
+    (pad "2" thru_hole oval (at 15.24 0 180) (size 3.2 3.2) (drill 1.6) (layers *.Cu *.Mask)
       (net 10 "Track3") (pinfunction "A") (pintype "passive"))
     (model "${KICAD6_3DMODEL_DIR}/Diode_THT.3dshapes/D_DO-201AD_P15.24mm_Horizontal.wrl"
@@
   )
   (footprint "Diode_THT:D_DO-201AD_P15.24mm_Horizontal" (layer "F.Cu")
-    (at 97.020225 85.76)
+    (at 50.8 15.24 180)
     (descr "Diode, DO-201AD series, Axial, Horizontal, pin pitch=15.24mm, , length*diameter=9.5*5.2mm^2, , http://www.diodes.com/_files/packages/DO-201AD.pdf")
     (tags "Diode DO-201AD series Axial Horizontal pin pitch 15.24mm  length 9.5mm diameter 5.2mm")
@@
     (fp_line (start 4.395 -2.6) (end 4.395 2.6) (layer "F.Fab") (width 0.1))
     (fp_line (start 2.87 -2.6) (end 2.87 2.6) (layer "F.Fab") (width 0.1))
-    (pad "1" thru_hole rect (at 0 0) (size 3.2 3.2) (drill 1.6) (layers *.Cu *.Mask)
+    (pad "1" thru_hole rect (at 0 0 180) (size 3.2 3.2) (drill 1.6) (layers *.Cu *.Mask)
       (net 2 "Dcc2") (pinfunction "K") (pintype "passive"))
-    (pad "2" thru_hole oval (at 15.24 0) (size 3.2 3.2) (drill 1.6) (layers *.Cu *.Mask)
+    (pad "2" thru_hole oval (at 15.24 0 180) (size 3.2 3.2) (drill 1.6) (layers *.Cu *.Mask)
       (net 7 "Net-(D1-Pad2)") (pinfunction "A") (pintype "passive"))
     (model "${KICAD6_3DMODEL_DIR}/Diode_THT.3dshapes/D_DO-201AD_P15.24mm_Horizontal.wrl"
@@
     (property "Sheetname" "")
     (attr through_hole)
-    (fp_text reference "R120" (at 2.54 -1.92) (layer "F.SilkS")
+    (fp_text reference "R120" (at -51.300225 -24.98) (layer "F.SilkS")
       (effects (font (size 1 1) (thickness 0.15)))
     )
@@
   )
   (footprint "Diode_THT:D_DO-201AD_P15.24mm_Horizontal" (layer "F.Cu")
-    (at 97.020225 99.26)
+    (at 43.18 76.2)
     (descr "Diode, DO-201AD series, Axial, Horizontal, pin pitch=15.24mm, , length*diameter=9.5*5.2mm^2, , http://www.diodes.com/_files/packages/DO-201AD.pdf")
     (tags "Diode DO-201AD series Axial Horizontal pin pitch 15.24mm  length 9.5mm diameter 5.2mm")
@@
   )
   (footprint "Diode_THT:D_DO-201AD_P15.24mm_Horizontal" (layer "F.Cu")
-    (at 43.18 27.94)
+    (at 38.1 35.56)
     (descr "Diode, DO-201AD series, Axial, Horizontal, pin pitch=15.24mm, , length*diameter=9.5*5.2mm^2, , http://www.diodes.com/_files/packages/DO-201AD.pdf")
     (tags "Diode DO-201AD series Axial Horizontal pin pitch 15.24mm  length 9.5mm diameter 5.2mm")
@@
   )
   (footprint "Diode_THT:D_DO-201AD_P15.24mm_Horizontal" (layer "F.Cu")
-    (at 154.080225 63.36)
+    (at 35.56 20.32)
     (descr "Diode, DO-201AD series, Axial, Horizontal, pin pitch=15.24mm, , length*diameter=9.5*5.2mm^2, , http://www.diodes.com/_files/packages/DO-201AD.pdf")
     (tags "Diode DO-201AD series Axial Horizontal pin pitch 15.24mm  length 9.5mm diameter 5.2mm")
@@
   )
   (footprint "Diode_THT:D_DO-201AD_P15.24mm_Horizontal" (layer "F.Cu")
-    (at 97.020225 68.92)
+    (at 53.34 30.48 180)
     (descr "Diode, DO-201AD series, Axial, Horizontal, pin pitch=15.24mm, , length*diameter=9.5*5.2mm^2, , http://www.diodes.com/_files/packages/DO-201AD.pdf")
     (tags "Diode DO-201AD series Axial Horizontal pin pitch 15.24mm  length 9.5mm diameter 5.2mm")
@@
     (fp_line (start 2.87 2.6) (end 12.37 2.6) (layer "F.Fab") (width 0.1))
     (fp_line (start 12.37 -2.6) (end 2.87 -2.6) (layer "F.Fab") (width 0.1))
-    (pad "1" thru_hole rect (at 0 0) (size 3.2 3.2) (drill 1.6) (layers *.Cu *.Mask)
+    (pad "1" thru_hole rect (at 0 0 180) (size 3.2 3.2) (drill 1.6) (layers *.Cu *.Mask)
       (net 7 "Net-(D1-Pad2)") (pinfunction "K") (pintype "passive"))
-    (pad "2" thru_hole oval (at 15.24 0) (size 3.2 3.2) (drill 1.6) (layers *.Cu *.Mask)
+    (pad "2" thru_hole oval (at 15.24 0 180) (size 3.2 3.2) (drill 1.6) (layers *.Cu *.Mask)
       (net 9 "Track2") (pinfunction "A") (pintype "passive"))
     (model "${KICAD6_3DMODEL_DIR}/Diode_THT.3dshapes/D_DO-201AD_P15.24mm_Horizontal.wrl"
